File: Electrical/Dyno_LED_PCB/Dyno_LED_PCB.kicad_sch (KiCad schematic)
At the start: 14 parts, among them J1 Conn_01x02, J2 Conn_01x02

Commit message: rev 2 circuit basically done, board almost laid out, also mechanical updates
Parts:
- C1, C2: value C_Polarized_Small -> 100u
Changed lines of the file:
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@@
 (kicad_sch
-	(version 20231120)
+	(version 20250114)
 	(generator "eeschema")
-	(generator_version "8.0")
+	(generator_version "9.0")
 	(paper "A4")
 	(junction
@@
 			)
 		)
-		(property "Value" "C_Polarized_Small"
+		(property "Value" "100u"
 			(at 106.68 74.3838 0)
 			(effects
@@
 			)
 		)
-		(property "Value" "C_Polarized_Small"
+		(property "Value" "100u"
 			(at 106.68 87.0838 0)
 			(effects
@@
 		)
 	)
+	(embedded_fonts no)
 )
